File: pcb/pcb.kicad_pcb (KiCad board)
At the start: 2 copper layers, 59 x 69 mm, 18 parts, among them J1 Screw_Terminal_01x02, J2 Screw_Terminal_01x03, J3 Screw_Terminal_01x03, J4 Conn_01x03_Pin, Q1 BUZ11, Q2 BUZ11, Q3 BUZ11, Q4 BUZ11, U1 L7805

Commit message: fix pcb issues
Parts:
- removed R1, R2, R3, R4: 10k, Resistor_SMD:R_1206_3216Metric_Pad1.30x1.75mm_HandSolder
- Q1, Q2, Q3, Q4: footprint Package_TO_SOT_THT:TO-220-3_Vertical -> Package_TO_SOT_THT:TO-220-3_Horizontal_TabDown
- U1: footprint Package_TO_SOT_THT:TO-220-3_Vertical -> Package_TO_SOT_THT:TO-220-3_Horizontal_TabUp
- moved J4 33.6 mm to (137.0, 106.5), turned to 180 degrees
- moved Q1 22.1 mm to (123.0, 102.2), turned to 0 degrees
- moved Q3 19.5 mm to (112.0, 102.2), turned to 0 degrees
- moved Q2 16.4 mm to (123.0, 79.2)
- moved Q4 14.2 mm to (112.0, 79.2)
- moved U1 14.0 mm to (133.5, 63.0), turned to 0 degrees
Connections:
- Q1 pad 2: GND -> GND_WW1
- Q1 pad 3: GND_WW1 -> GND
- Q2 pad 2: GND -> GND_CW1
- Q2 pad 3: GND_CW1 -> GND
- Q3 pad 2: GND -> GND_WW2
- Q3 pad 3: GND_WW2 -> GND
- Q4 pad 2: GND -> GND_CW2
- Q4 pad 3: GND_CW2 -> GND
Routing:
- net +5V: track 32.9 -> 80.7 mm
- net PWM_SERVO: track 35.2 -> 64.0 mm
- net PWM_WW_CENTER: track 42.2 -> 17.9 mm
- net GND_WW1: track 29.4 -> 10.0 mm
- net GND_WW2: track 28.8 -> 11.1 mm
- net PWM_CW_CENTER: track 35.5 -> 52.2 mm
- net GND_CW2: track 21.6 -> 37.1 mm
- net +12V: track 93.6 -> 78.3 mm
- net GND: track 29.8 -> 15.1 mm, vias 13 -> 1
- net GND_CW1: track 22.2 -> 36.1 mm
- net PWM_WW_RING: track 23.5 -> 9.96 mm
- net PWM_CW_RING: track 16.3 -> 20.5 mm
Other:
- board text added: "12V"
- board text added: "5V"
- board text added: "PWM"
- board text removed: "+12V"
