File: pcb/pcb.kicad_sch (KiCad schematic)
At the start: 18 parts, among them J1 Screw_Terminal_01x02, J2 Screw_Terminal_01x03, J3 Screw_Terminal_01x03, J4 Conn_01x03_Pin, Q1 BUZ11, Q2 BUZ11, Q3 BUZ11, Q4 BUZ11, U1 L7805

Commit message: fix pcb issues
Parts:
- removed R1, R2, R3, R4: 10k, Resistor_SMD:R_1206_3216Metric_Pad1.30x1.75mm_HandSolder, symbol Device:R
- Q1, Q2, Q3, Q4: footprint Package_TO_SOT_THT:TO-220-3_Vertical -> Package_TO_SOT_THT:TO-220-3_Horizontal_TabDown
- U1: footprint Package_TO_SOT_THT:TO-220-3_Vertical -> Package_TO_SOT_THT:TO-220-3_Horizontal_TabUp
Connections:
- net GND: now also Q1.3 (S), Q2.3 (S), Q3.3 (S), Q4.3 (S); no longer Q1.2 (D), Q2.2 (D), Q3.2 (D), Q4.2 (D)
- net GND_CW1: now also Q2.2 (D); no longer Q2.3 (S)
- net GND_CW2: now also Q4.2 (D); no longer Q4.3 (S)
- net GND_WW1: now also Q1.2 (D); no longer Q1.3 (S)
- net GND_WW2: now also Q3.2 (D); no longer Q3.3 (S)
Other:
- moved on the sheet: Q1, Q2, Q3, Q4
